Commit message: change the size and location of spawned cubes

File: ros/collab_ws/src/collaborative_robotics_course/locobot_autonomy/model/blue_cube.urdf (robot description, URDF)
Before this commit: robot blue_cube, 1 links, 0 joints
Links:
- link my_box: geometry collision box size=0.2 0.2 0.2; visual box size=0.2 0.2 0.2

File: ros/collab_ws/src/collaborative_robotics_course/locobot_autonomy/model/red_cube.urdf (robot description, URDF)
Before this commit: robot red_cube, 1 links, 0 joints
Links:
- link my_box: geometry collision box size=0.2 0.2 0.2; visual box size=0.2 0.2 0.2

File: ros/collab_ws/src/collaborative_robotics_course/locobot_autonomy/model/yellow_cube.urdf (robot description, URDF)
Before this commit: robot yellow_cube, 1 links, 0 joints
Links:
- link my_box: geometry collision box size=0.2 0.2 0.2; visual box size=0.2 0.2 0.2
